Commit message: new urdf

File: auto_nav/urdf/sensors_orchards.xacro (robot description, xacro)
@@ -15,5 +15,5 @@
     <parent link="$(arg tf_prefix)/base_link"/>
     <child link="$(arg tf_prefix)/gps"/>
-    <origin xyz="0.425 -0.62 1.05"/>
+    <origin xyz="0.425 -0.766 1.05"/>
   </joint>
   <!--IMU-->
@@ -29,5 +29,5 @@
     <parent link="$(arg tf_prefix)/base_link"/>
     <child link="$(arg tf_prefix)/xsens"/>
-    <origin xyz="0.385 0.0 0.8" rpy="0 0 0"/>
+    <origin xyz="0.350 0.0 0.765" rpy="0 0 0"/>
   </joint>
   <!--Basler-->
@@ -82,5 +82,5 @@
       <parent link="$(arg tf_prefix)/base_link"/>
       <child link="$(arg tf_prefix)/camera_bottom_screw_frame" />
-      <origin xyz="0.815 0.0 1.115" rpy="0 0.0 0" />
+      <origin xyz="0.845 0.0 1.09" rpy="0 0.1745 0" />
     </joint>
     <link name="$(arg tf_prefix)/camera_link">

Commit message: updates

File: auto_nav/urdf/sensors_orchards.xacro (robot description, xacro)
@@ -82,5 +82,5 @@
       <parent link="$(arg tf_prefix)/base_link"/>
       <child link="$(arg tf_prefix)/camera_bottom_screw_frame" />
-      <origin xyz="0.845 0.0 1.09" rpy="0 0.1745 0" />
+      <origin xyz="0.845 0.0 1.09" rpy="0 0.2620 0" />
     </joint>
     <link name="$(arg tf_prefix)/camera_link">
