Commit message: Basler and flir Camera Links added in Tf frame.

File: auto_nav/urdf/sensors_frogn.xacro (robot description, xacro)
@@ -30,4 +30,28 @@
     <child link="$(arg tf_prefix)/xsens"/>
     <origin xyz="0.31 0.0 0.8" rpy="0 0 0"/>
+  </joint>
+  <!--Basler-->
+  <!-- camera body, with origin at bottom screw mount -->
+  <link name="$(arg tf_prefix)/basler_camera"/>
+  <joint name="basler_camera_joint" type="fixed">
+    <parent link="$(arg tf_prefix)/base_link"/>
+    <child link="$(arg tf_prefix)/basler_camera" />
+    <origin xyz="0.735 0.0 1.205" rpy="0 0.366519 0" />
+  </joint>
+  <!--FLIR Camera 1-->
+  <!-- camera body, with origin at bottom screw mount -->
+  <link name="$(arg tf_prefix)/flir_camera_1"/>
+  <joint name="flir_camera_1_joint" type="fixed">
+    <parent link="$(arg tf_prefix)/base_link"/>
+    <child link="$(arg tf_prefix)/flir_camera_1" />
+    <origin xyz="0.735 -0.1 1.205" rpy="0 0.366519 0" />
+  </joint>
+  <!--FLIR Camera 2-->
+  <!-- camera body, with origin at bottom screw mount -->
+  <link name="$(arg tf_prefix)/flir_camera_2"/>
+  <joint name="flir_camera_2_joint" type="fixed">
+    <parent link="$(arg tf_prefix)/base_link"/>
+    <child link="$(arg tf_prefix)/flir_camera_2" />
+    <origin xyz="0.735 0.1 1.205" rpy="0 0.366519 0" />
   </joint>
   <!--Camera-->

Commit message: lastst NUC

File: auto_nav/urdf/sensors_frogn.xacro (robot description, xacro)
@@ -37,5 +37,5 @@
     <parent link="$(arg tf_prefix)/base_link"/>
     <child link="$(arg tf_prefix)/basler_camera" />
-    <origin xyz="0.735 0.0 1.205" rpy="0 0.366519 0" />
+    <origin xyz="0.75 0.0 1.055" rpy="0 0.279253 0" />
   </joint>
   <!--FLIR Camera 1-->
@@ -45,5 +45,5 @@
     <parent link="$(arg tf_prefix)/base_link"/>
     <child link="$(arg tf_prefix)/flir_camera_1" />
-    <origin xyz="0.735 -0.1 1.205" rpy="0 0.366519 0" />
+    <origin xyz="0.75 0.22 1.055" rpy="0 0.279253 0" />
   </joint>
   <!--FLIR Camera 2-->
@@ -53,5 +53,5 @@
     <parent link="$(arg tf_prefix)/base_link"/>
     <child link="$(arg tf_prefix)/flir_camera_2" />
-    <origin xyz="0.735 0.1 1.205" rpy="0 0.366519 0" />
+    <origin xyz="0.75 -0.21 1.055" rpy="0 0.279253 0" />
   </joint>
   <!--Camera-->

Commit message: urdf and ekf updates

File: auto_nav/urdf/sensors_frogn.xacro (robot description, xacro)
@@ -15,5 +15,5 @@
     <parent link="$(arg tf_prefix)/base_link"/>
     <child link="$(arg tf_prefix)/gps"/>
-    <origin xyz="0.425 -0.62 1.05"/>
+    <origin xyz="0.425 -0.625 1.05"/>
   </joint>
   <!--IMU-->
@@ -29,5 +29,5 @@
     <parent link="$(arg tf_prefix)/base_link"/>
     <child link="$(arg tf_prefix)/xsens"/>
-    <origin xyz="0.31 0.0 0.8" rpy="0 0 0"/>
+    <origin xyz="0.315 0.0 0.8" rpy="0 0 0"/>
   </joint>
   <!--Basler-->
@@ -82,5 +82,5 @@
       <parent link="$(arg tf_prefix)/base_link"/>
       <child link="$(arg tf_prefix)/camera_bottom_screw_frame" />
-      <origin xyz="0.745 0.0 1.230" rpy="0 0.331613 0" />
+      <origin xyz="0.855 0.0 1.230" rpy="0 0.331613 0" />
     </joint>
     <link name="$(arg tf_prefix)/camera_link">

Commit message: correct eccentrifities

File: auto_nav/urdf/sensors_frogn.xacro (robot description, xacro)
@@ -15,5 +15,5 @@
     <parent link="$(arg tf_prefix)/base_link"/>
     <child link="$(arg tf_prefix)/gps"/>
-    <origin xyz="0.425 -0.625 1.05"/>
+    <origin xyz="0.4155 -0.1615 1.0130"/>
   </joint>
   <!--IMU-->
@@ -29,5 +29,5 @@
     <parent link="$(arg tf_prefix)/base_link"/>
     <child link="$(arg tf_prefix)/xsens"/>
-    <origin xyz="0.315 0.0 0.8" rpy="0 0 0"/>
+    <origin xyz="0.3500 -0.0183 0.8070" rpy="0 0 0"/>
   </joint>
   <!--Basler-->
@@ -37,5 +37,5 @@
     <parent link="$(arg tf_prefix)/base_link"/>
     <child link="$(arg tf_prefix)/basler_camera" />
-    <origin xyz="0.735 0.0 1.055" rpy="0 0.3926991 0" />
+    <origin xyz="0.8475 0.0005 1.0640" rpy="0 0.3787 0" />
   </joint>
   <!--FLIR Camera 1-->
@@ -45,5 +45,5 @@
     <parent link="$(arg tf_prefix)/base_link"/>
     <child link="$(arg tf_prefix)/flir_camera_1" />
-    <origin xyz="0.735 0.22 1.055" rpy="0 0.3926991 0" />
+    <origin xyz="0.735 0.22 1.055" rpy="0 0.367 0" />
   </joint>
   <!--FLIR Camera 2-->
@@ -53,5 +53,5 @@
     <parent link="$(arg tf_prefix)/base_link"/>
     <child link="$(arg tf_prefix)/flir_camera_2" />
-    <origin xyz="0.735 -0.21 1.055" rpy="0 0.3926991 0" />
+    <origin xyz="0.735 -0.21 1.055" rpy="0 0.367 0" />
   </joint>
   <!--Camera-->
@@ -82,5 +82,5 @@
       <parent link="$(arg tf_prefix)/base_link"/>
       <child link="$(arg tf_prefix)/camera_bottom_screw_frame" />
-      <origin xyz="0.855 0.0 1.230" rpy="0 0.331613 0" />
+      <origin xyz="0.8045 0.0035 0.9920" rpy="0 0.2942 0" />
     </joint>
     <link name="$(arg tf_prefix)/camera_link">

Commit message: eccentrities

File: auto_nav/urdf/sensors_frogn.xacro (robot description, xacro)
@@ -26,10 +26,10 @@
     <parent link="$(arg tf_prefix)/base_link"/>
     <child link="$(arg tf_prefix)/septentrio"/>
-    <origin xyz="0.8045 0.28 1.1" rpy="0 0 0"/>
+    <origin xyz="0.7657 -0.2795 1.0828" rpy="0 0 0"/>
   </joint>
   <joint name="$(arg tf_prefix)/base_septentrio_static2" type="fixed">
     <parent link="$(arg tf_prefix)/base_link"/>
     <child link="$(arg tf_prefix)/septentrio_static2"/>
-    <origin xyz="0.8045 -0.28 1.1" rpy="0 0 0"/>
+    <origin xyz="0.7657 0.2795 1.0828" rpy="0 0 0"/>
   </joint>
   <!--GNSS-->
@@ -112,5 +112,5 @@
       <parent link="$(arg tf_prefix)/base_link"/>
       <child link="$(arg tf_prefix)/camera_bottom_screw_frame" />
-      <origin xyz="0.8045 0.0035 0.9920" rpy="0 0.2942 0" />
+      <origin xyz="0.8118 0.0035 1.0729" rpy="0 0.2942 0" />
     </joint>
     <link name="$(arg tf_prefix)/camera_link">
